Commit message: Model parameter estimation generic Move evaluation to dlkineamtics package Fix model parameter estimation example

File: data/random_chain_2.urdf (robot description, URDF)
Before this commit: robot chain6, 7 links, 6 joints
Links:
- removed link link3
- removed link link4
- removed link link5
- removed link link6
Joints:
- removed joint joint2
- removed joint joint3
- removed joint joint4
- removed joint joint5
- joint joint0: axis 0 0 1 -> 0 1 0; limit lower=-0.2994356447454922 upper=0.5372737659974582 effort=0.0 velocity=0.0 -> lower=-0.7467977126727877 upper=1.634520136596924 effort=0.0 velocity=0.0; origin xyz=0.39 -0.00 -0.31 rpy=2.33 -0.20 -0.53 -> xyz=0.67 -0.78 -0.11 rpy=1.56 2.50 -1.87; type prismatic -> revolute
- joint joint1: limit lower=-2.1177220741313763 upper=1.7734052709900225 effort=0.0 velocity=0.0 -> lower=-0.409708700339666 upper=0.19606005240497826 effort=0.0 velocity=0.0; origin xyz=-0.49 0.40 -0.14 rpy=0.90 2.11 -0.36 -> xyz=1.61 -1.40 -0.73 rpy=0.21 -0.01 0.03; type revolute -> prismatic

File: data/random_chain_6.urdf (robot description, URDF)
Before this commit: robot chain6, 7 links, 6 joints
Joints:
- joint joint0: axis 1 0 0 -> 0 1 0; limit (none) -> lower=-0.6939597249482587 upper=0.49741024074612594 effort=0.0 velocity=0.0; origin xyz=1.56 -0.43 -1.01 rpy=3.03 -2.57 -0.30 -> xyz=-1.65 0.15 -1.99 rpy=-0.07 1.17 2.16
- joint joint1: axis 0 1 0 -> 1 0 0; limit (none) -> lower=-1.2323281494491418 upper=2.9138689589681546 effort=0.0 velocity=0.0; origin xyz=1.14 -1.34 0.56 rpy=-1.41 -0.30 -0.15 -> xyz=-1.74 -1.26 -1.93 rpy=2.98 1.18 1.66
- joint joint2: axis 0 0 1 -> 0 1 0; limit (none) -> lower=-0.16045891452798122 upper=0.8482404436144259 effort=0.0 velocity=0.0; origin xyz=0.96 -0.11 -1.14 rpy=1.42 -0.30 0.77 -> xyz=-1.75 -1.18 0.28 rpy=2.25 2.64 -0.30
- joint joint3: limit (none) -> effort=0.0 velocity=0.0; origin xyz=-1.41 -0.08 1.51 rpy=-2.62 -2.07 2.97 -> xyz=0.57 0.75 -1.04 rpy=1.86 -2.70 -2.22; type prismatic -> continuous
- joint joint4: axis 1 0 0 -> 0 1 0; limit (none) -> effort=0.0 velocity=0.0; origin xyz=1.79 0.94 1.56 rpy=0.28 -2.27 -2.45 -> xyz=0.83 -1.22 -1.94 rpy=0.86 1.17 0.58; type prismatic -> continuous
- joint joint5: axis 1 0 0 -> 0 1 0; limit (none) -> lower=-0.6791673519998924 upper=0.32489354914652224 effort=0.0 velocity=0.0; origin xyz=1.00 1.33 1.40 rpy=1.24 -1.72 -3.08 -> xyz=-0.29 1.87 -1.45 rpy=1.58 -0.52 1.03; type revolute -> prismatic
